Commit message: added static transform node

File: urdf/lidarbot1.urdf.xacro (robot description, xacro)
@@ -5,4 +5,3 @@
     <xacro:include filename="depth_camera.xacro"/>
     <xacro:include filename="gazebo_control.xacro"/>
-    <xacro:include filename="imu.xacro"/>
 </robot>

File: urdf/lidarbot1_core.xacro (robot description, xacro)
@@ -24,5 +24,4 @@
     </material>
     <link name="base_footprint"/>
-    <link name="base_link" />
     <link name="chassis_link">
         <visual>
@@ -116,11 +115,6 @@
     </gazebo>
     <!-- JOINTS -->
-    <joint name="base_link_joint" type="fixed">
-        <parent link="base_footprint" />
-        <child link="base_link" />
-        <origin xyz="0 0 0" rpy="0 0 0" />
-    </joint>
     <joint name="chassis_base_joint" type="fixed">
-        <parent link="base_link"/>
+        <parent link="base_footprint"/>
         <child link="chassis_link"/>
         <origin xyz="0 0 ${wheel_r}" rpy="0 0 0"/>
