Commit message: fixed bug 2: imu sensor not publishing data to /imu/data

File: urdf/imu.xacro (robot description, xacro)
@@ -4,83 +4,45 @@
     <parent link="chassis_link"/>
     <child link="imu_link"/>
-    <origin xyz="-0.10 0.1 0.05" rpy="0 0 0"/>
+    <origin xyz="0 0 0.2" rpy="0 0 0"/>
   </joint>
   <link name="imu_link">
+    <visual>
+        <geometry>
+            <box size="0.04 0.02 0.02"/>
+        </geometry>
+        <origin xyz="0 0 0"/>
+        <material name="green"/>
+    </visual>
+    <collision>
+        <geometry>
+            <box size="0.1 0.1 0.1"/>
+        </geometry>
+        <origin xyz="0 0 0"/>
+    </collision>
+    <inertial>
+        <mass value="2.0"/>
+        <inertia ixx="0.1" ixy="0" ixz="0" iyy="0.1" iyz="0" izz="0.1"/>
+    </inertial>
+  </link>
+  <gazebo reference="imu_link">
     <gravity>true</gravity>
-    <sensor name="bmb_imu" type="imu">
+    <sensor name="imu_sensor" type="imu">
       <always_on>true</always_on>
       <update_rate>100</update_rate>
       <visualize>true</visualize>
-      <imu>
-        <orientation>
-          <x>
-            <noise type="gaussian">
-              <mean>0.0</mean>
-              <stddev>2e-3</stddev>
-            </noise>
-          </x>
-          <y>
-            <noise type="gaussian">
-              <mean>0.0</mean>
-              <stddev>2e-3</stddev>
-            </noise>
-          </y>
-          <z>
-            <noise type="gaussian">
-              <mean>0.0</mean>
-              <stddev>2e-3</stddev>
-            </noise>
-          </z>
-        </orientation>
-        <angular_velocity>
-          <x>
-            <noise type="gaussian">
-              <mean>0.0</mean>
-              <stddev>2e-4</stddev>
-            </noise>
-          </x>
-          <y>
-            <noise type="gaussian">
-              <mean>0.0</mean>
-              <stddev>2e-4</stddev>
-            </noise>
-          </y>
-          <z>
-            <noise type="gaussian">
-              <mean>0.0</mean>
-              <stddev>2e-4</stddev>
-            </noise>
-          </z>
-        </angular_velocity>
-        <linear_acceleration>
-          <x>
-            <noise type="gaussian">
-              <mean>0.0</mean>
-              <stddev>1.7e-2</stddev>
-            </noise>
-          </x>
-          <y>
-            <noise type="gaussian">
-              <mean>0.0</mean>
-              <stddev>1.7e-2</stddev>
-            </noise>
-          </y>
-          <z>
-            <noise type="gaussian">
-              <mean>0.0</mean>
-              <stddev>1.7e-2</stddev>
-            </noise>
-          </z>
-        </linear_acceleration>
-      </imu>
-      <plugin name="imu_sensor" filename="libgazebo_ros_imu_sensor.so">
-        <initial_orientation_as_reference>false</initial_orientation_as_reference>
-        <frame_name>imu_link</frame_name>
-        <ros>
-          <namespace>/imu</namespace>
-          <remapping>~/out:=data</remapping>
-        </ros>
+      <topic>__default_topic__</topic>
+      <plugin filename="libgazebo_ros_imu_sensor.so" name="imu_plugin">
+        <topicName>imu</topicName>
+        <namespace>/</namespace>
+        <remapping>imu_plugin/out:=imu/data</remapping>
+        <bodyName>imu_link</bodyName>
+        <updateRateHZ>10.0</updateRateHZ>
+        <gaussianNoise>0.0</gaussianNoise>
+        <xyzOffset>0 0 0</xyzOffset>
+        <rpyOffset>0 0 0</rpyOffset>
+        <frameName>imu_link</frameName>
       </plugin>
+      <pose>0 0 0 0 0 0</pose>
     </sensor>
-  </link>
+  </gazebo>
 </robot>

File: urdf/lidarbot1.urdf.xacro (robot description, xacro)
@@ -3,9 +3,7 @@
     <xacro:include filename="lidarbot1_core.xacro"/>
     <xacro:include filename="lidar.xacro"/>
-    <!-- <xacro:include filename="camera.xacro"/> -->
     <xacro:include filename="depth_camera.xacro"/>
     <xacro:include filename="gazebo_control.xacro"/>
-    <!-- <xacro:include filename="ros2_control.xacro"/> -->
+    <xacro:include filename="ros2_control.xacro"/>
     <xacro:include filename="imu.xacro"/>
-    <!-- run odom_unfiltered, with tf2_broadcaster, with use_sim_time to false -->
 </robot>

Commit message: Fixed Bug 4: Navigation not working due to offset in base_footprint

File: urdf/imu.xacro (robot description, xacro)
@@ -33,13 +33,13 @@
       <topic>__default_topic__</topic>
       <plugin filename="libgazebo_ros_imu_sensor.so" name="imu_plugin">
-        <topicName>imu</topicName>
+        <topic_name>imu</topic_name>
         <namespace>/</namespace>
         <remapping>imu_plugin/out:=imu/data</remapping>
-        <bodyName>imu_link</bodyName>
-        <updateRateHZ>10.0</updateRateHZ>
-        <gaussianNoise>0.0</gaussianNoise>
-        <xyzOffset>0 0 0</xyzOffset>
-        <rpyOffset>0 0 0</rpyOffset>
-        <frameName>imu_link</frameName>
+        <body_name>imu_link</body_name>
+        <update_rate_hz>10.0</update_rate_hz>
+        <gaussian_noise>0.0</gaussian_noise>
+        <xyz_offset>0 0 0</xyz_offset>
+        <rpy_offset>0 0 0</rpy_offset>
+        <frame_name>imu_link</frame_name>
       </plugin>
       <pose>0 0 0 0 0 0</pose>

File: urdf/lidarbot1.urdf.xacro (robot description, xacro)
@@ -3,5 +3,5 @@
     <xacro:include filename="lidarbot1_core.xacro"/>
     <xacro:include filename="lidar.xacro"/>
-    <xacro:include filename="depth_camera.xacro"/>
+    <xacro:include filename="imu.xacro"/>
     <xacro:include filename="gazebo_control.xacro"/>
 </robot>

File: urdf/lidarbot1_core.xacro (robot description, xacro)
@@ -118,5 +118,5 @@
         <parent link="base_footprint"/>
         <child link="chassis_link"/>
-        <origin xyz="0 0 ${wheel_r}" rpy="0 0 0"/>
+        <origin xyz="0.15 0 ${wheel_r}" rpy="0 0 0"/>
     </joint>
     <joint name="left_wheel_chassis_joint" type="continuous">

File: urdf/ros2_control.xacro (robot description, xacro)
@@ -1,5 +1,5 @@
 <?xml version="1.0"?>
 <robot xmlns:xacro="http://www.ros.org/wiki/xacro">
-    <!-- <ros2_control name="GazeboSystem" type="System">
+    <ros2_control name="GazeboSystem" type="System">
         <hardware>
             <plugin>gazebo_ros2_control/GazeboSystem</plugin>
@@ -26,4 +26,4 @@
             <parameters>/home/user/ros2_ws/src/lidarbot1/config/controllers.yaml</parameters>
         </plugin>
-    </gazebo> -->
+    </gazebo>
 </robot>
